File: can_fet_conn_mre_wbo2.sch (KiCad schematic (older format))
At the start: 12 parts, among them J10 Molex_Micro-Fit_3.0_43045-060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, J20 Conn_02x05_Odd_Even-Connector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, J30 Conn_02x05_Odd_Even-Connector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, Q1 BTS3028, U5 TJA1051T-3

Commit message: Add files via upload
Parts:
- added C42: 100nF, Capacitor_SMD:C_0603_1608Metric, symbol micro_rusEFI-rescue:C-Device
- added J14: microSD_HC_Wuerth_693072010801, Connector_Card:microSD_HC_Wuerth_693072010801, symbol micro_rusEFI-rescue:Micro_SD_Card-Connector-proteus-rescue
Connections:
- wire segments 41 -> 51
- no-connect marks 10 -> 8
Other:
- moved on the sheet: F1, J10, J20

Commit message: Add files via upload
Parts:
- added C1101: 10nF, Capacitor_SMD:C_0603_1608Metric, symbol Device:C
- added C1102: 100nF, Capacitor_SMD:C_0603_1608Metric, symbol Device:C
- added J1: Soldering PAD for 12V_MREL, Connector_PinHeader_2.54mm:PinHeader_1x01_P2.54mm_Vertical, symbol Connector:Conn_01x01_Female
- added J40: CONN_Molex, Connector_Molex:Molex_Micro-Fit_3.0_43045-0200_2x01_P3.00mm_Horizontal, symbol Connector:Conn_01x02_Male
- added P1104: CONN_Sparkfun, rusefi_lib:tcpl_PCC-SMP, symbol Connector:Conn_01x02_Female
- added U1101: MAX31855KASA, Package_SO:SO-8_5.3x6.2mm_P1.27mm, symbol MAX31855KASA:MAX31855
- C42: symbol micro_rusEFI-rescue:C-Device -> wideband_controller_mre-rescue:C-Device-micro_rusEFI-rescue
- J10: symbol wideband_controller_mre-rescue:Conn_Molex_02x03 -> wideband_controller_mre-rescue:Conn_Molex_02x03-wideband_controller_mre-rescue
- J14: symbol micro_rusEFI-rescue:Micro_SD_Card-Connector-proteus-rescue -> wideband_controller_mre-rescue:Micro_SD_Card-Connector-proteus-rescue-micro_rusEFI-rescue
- J20, J30: symbol wideband_controller_mre-rescue:Conn_02x05_Odd_Even-Connector_Generic -> wideband_controller_mre-rescue:Conn_02x05_Odd_Even-Connector_Generic-wideband_controller_mre-rescue
- U5: symbol can_conn_mre_wbo2-rescue:TJA1051T-3-Interface_CAN_LIN -> wideband_controller_mre-rescue:TJA1051T-3-Interface_CAN_LIN-can_conn_mre_wbo2-rescue
Connections:
- net labels added: TCPL+, TCPL-
- wire segments 51 -> 62
Other:
- note added: "Datasheet:\nhttp://datasheets.maxim-ic.com/en/ds/MAX31855.pdf"
- note added: "MAX31855\nCold-Junction Compensated\nThermocouple-to-Digital Converter"
- moved on the sheet: C23, C24, C42, D1, F1, J10, J15, J20, J30, Q1, R32, R33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
