File: can_fet_conn_mre_wbo2.sch (KiCad schematic (older format))
At the start: 20 parts, among them J1 Soldering PAD for 12V_MREL, J10 Molex_Micro-Fit_3.0_43045-060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, J14 microSD_HC_Wuerth_693072010801, J20 Conn_02x05_Odd_Even-Connector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, J30 Conn_02x05_Odd_Even-Connector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, J40 CONN_Molex, P1104 CONN_Sparkfun, Q1 BTS3028, U1101 MAX31855KASA, U5 TJA1051T-3

Commit message: Add files via upload
Parts:
- added C21: 100nF, Capacitor_SMD:C_0603_1608Metric, symbol wideband_controller_mre-rescue:C-Device-micro_rusEFI-rescue
- renumbered J1 to J21
Connections:
- wire segments 62 -> 64
Changed lines of the file:
@@
 Text GLabel 10100 1450 2    50   Input ~ 0
 LSU_Un
-Text GLabel 4200 2100 0    50   Input ~ 0
+Text GLabel 5950 2850 0    50   Input ~ 0
 +5V
-Text GLabel 4200 2250 0    50   Input ~ 0
+Text GLabel 5950 3000 0    50   Input ~ 0
 +3.3V
 $Comp
 L Power:+3.3V #PWR0111
 U 1 1 61992392
-P 4525 2250
-F 0 "#PWR0111" H 4525 2100 50  0001 C CNN
-F 1 "+3.3V" V 4540 2378 50  0000 L CNN
-F 2 "" H 4525 2250 50  0001 C CNN
-F 3 "" H 4525 2250 50  0001 C CNN
-	1    4525 2250
+P 6275 3000
+F 0 "#PWR0111" H 6275 2850 50  0001 C CNN
+F 1 "+3.3V" V 6290 3128 50  0000 L CNN
+F 2 "" H 6275 3000 50  0001 C CNN
+F 3 "" H 6275 3000 50  0001 C CNN
+	1    6275 3000
 	0    1    1    0
 $EndComp
@@
 L Power:+5V #PWR0112
 U 1 1 61992A8F
-P 4525 2100
-F 0 "#PWR0112" H 4525 1950 50  0001 C CNN
-F 1 "+5V" V 4540 2228 50  0000 L CNN
-F 2 "" H 4525 2100 50  0001 C CNN
-F 3 "" H 4525 2100 50  0001 C CNN
-	1    4525 2100
+P 6275 2850
+F 0 "#PWR0112" H 6275 2700 50  0001 C CNN
+F 1 "+5V" V 6290 2978 50  0000 L CNN
+F 2 "" H 6275 2850 50  0001 C CNN
+F 3 "" H 6275 2850 50  0001 C CNN
+	1    6275 2850
 	0    1    1    0
 $EndComp
 Wire Wire Line
-	4200 2250 4525 2250
+	5950 3000 6275 3000
 Text GLabel 1325 1650 0    50   Input ~ 0
 CAN_TX
@@
 Wire Wire Line
 	1325 1750 1825 1750
-Text GLabel 4200 2400 0    50   Input ~ 0
+Text GLabel 5950 3150 0    50   Input ~ 0
 GND
 $Comp
 L Power:GND #PWR0123
 U 1 1 61A069D4
-P 4525 2400
-F 0 "#PWR0123" H 4525 2150 50  0001 C CNN
-F 1 "GND" V 4530 2272 50  0000 R CNN
-F 2 "" H 4525 2400 50  0001 C CNN
-F 3 "" H 4525 2400 50  0001 C CNN
-	1    4525 2400
+P 6275 3150
+F 0 "#PWR0123" H 6275 2900 50  0001 C CNN
+F 1 "GND" V 6280 3022 50  0000 R CNN
+F 2 "" H 6275 3150 50  0001 C CNN
+F 3 "" H 6275 3150 50  0001 C CNN
+	1    6275 3150
 	0    -1   -1   0
 $EndComp
 Wire Wire Line
-	4200 2400 4525 2400
+	5950 3150 6275 3150
 $Comp
 L Power:+3.3V #PWR0148
@@
 $EndComp
 Wire Wire Line
-	4200 2100 4525 2100
+	5950 2850 6275 2850
 Text Label 9600 2575 0    50   ~ 0
 5V
@@
 $EndComp
 $Comp
-L Connector:Conn_01x01_Female J1
+L Connector:Conn_01x01_Female J21
 U 1 1 619E5055
 P 9600 2150
-F 0 "J1" H 9628 2176 50  0000 L CNN
+F 0 "J21" H 9628 2176 50  0000 L CNN
 F 1 "Soldering PAD for 12V_MREL" H 9628 2085 50  0000 L CNN
 F 2 "Connector_PinHeader_2.54mm:PinHeader_1x01_P2.54mm_Vertical" H 9600 2150 50  0001 C CNN
@@
 Wire Wire Line
 	9025 2150 9400 2150
+$Comp
+L wideband_controller_mre-rescue:C-Device-micro_rusEFI-rescue C21
+U 1 1 619F64D5
+P 4200 2075
+F 0 "C21" H 4315 2121 50  0000 L CNN
+F 1 "100nF" H 4315 2030 50  0000 L CNN
+F 2 "Capacitor_SMD:C_0603_1608Metric" H 4238 1925 50  0001 C CNN
+F 3 "~" H 4200 2075 50  0001 C CNN
+F 4 "C0603C104J5RACTU" H -1800 150 50  0001 C CNN "Part #"
+F 5 "DIGI" H -1800 150 50  0001 C CNN "VEND"
+F 6 "399-7844-1-ND" H -1800 150 50  0001 C CNN "VEND#"
+F 7 "KEMET" H -1800 150 50  0001 C CNN "Manufacturer"
+F 8 "C14663" H 4200 2075 50  0001 C CNN "LCSC"
+	1    4200 2075
+	-1   0    0    1
+$EndComp
+$Comp
+L wideband_controller_mre-rescue:GND-power-micro_rusEFI-rescue #PWR0170
+U 1 1 619F64DB
+P 4200 2300
+F 0 "#PWR0170" H 4200 2050 50  0001 C CNN
+F 1 "GND" H 4205 2127 50  0000 C CNN
+F 2 "" H 4200 2300 50  0001 C CNN
+F 3 "" H 4200 2300 50  0001 C CNN
+	1    4200 2300
+	1    0    0    -1
+$EndComp
+Wire Wire Line
+	4200 1750 4200 1925
+Wire Wire Line
+	4200 2300 4200 2225
+Text Label 4200 1750 2    50   ~ 10
+5V
 $EndSCHEMATC

Commit message: Add files via upload
Parts:
- F1: footprint Resistor_SMD:R_1206_3216Metric -> Resistor_SMD:R_2816_7142Metric
Changed lines of the file:
@@
 Sheet 3 3
 Title "MRE addon board - WBO2 & EGT & SD Card"
-Date "2021-11-26"
+Date "2021-12-02"
 Rev "V1.3"
 Comp "by JRD McLAREN"
@@
 F 0 "F1" V 9525 1900 50  0000 C CNN
 F 1 "Polyfuse 2A" V 9434 1900 50  0000 C CNN
-F 2 "Resistor_SMD:R_1206_3216Metric" H 9350 1700 50  0001 L CNN
+F 2 "Resistor_SMD:R_2816_7142Metric" H 9350 1700 50  0001 L CNN
 F 3 "~" H 9300 1900 50  0001 C CNN
 	1    9300 1900
