File: mcu_adc_mre_wbo2.sch (KiCad schematic (older format))
At the start: 50 parts, among them J1 TC2030, J2 Conn_01x06_Male, J3 Conn_01x03_Male, SW1 SW_Push, U1 STM32F042K6Tx, U2 MCP6004, U3 AD8628, U4 REF3033

Commit message: Add files via upload
Parts:
- JP1, JP2: symbol wideband_controller_mre-rescue:Jumper_3_Open-Jumper -> wideband_controller_mre-rescue:Jumper_3_Open-Jumper-wideband_controller_mre-rescue
- U1: symbol wideband_controller_mre-rescue:STM32F042K6Tx-MCU_ST_STM32F0 -> wideband_controller_mre-rescue:STM32F042K6Tx-MCU_ST_STM32F0-wideband_controller_mre-rescue
- U2: symbol wideband_controller_mre-rescue:MCP6004-Amplifier_Operational -> wideband_controller_mre-rescue:MCP6004-Amplifier_Operational-wideband_controller_mre-rescue
- U3: symbol wideband_controller_mre-rescue:AD8603-Amplifier_Operational -> wideband_controller_mre-rescue:AD8603-Amplifier_Operational-wideband_controller_mre-rescue
- U4: symbol wideband_controller_mre-rescue:REF3033-Reference_Voltage -> wideband_controller_mre-rescue:REF3033-Reference_Voltage-wideband_controller_mre-rescue
Changed lines of the file:
@@
 $EndComp
 $Comp
-L wideband_controller_mre-rescue:GND-power #PWR0102
+L wideband_controller_mre-rescue:GND-power-wideband_controller_mre-rescue #PWR0102
 U 1 1 5EB10275
 P 1100 1675
@@
 	800  1275 1100 1275
 $Comp
-L wideband_controller_mre-rescue:GND-power #PWR0103
+L wideband_controller_mre-rescue:GND-power-wideband_controller_mre-rescue #PWR0103
 U 1 1 5EB130B2
 P 800 1675
@@
 	4700 1375 4600 1375
 $Comp
-L wideband_controller_mre-rescue:GND-power #PWR0104
+L wideband_controller_mre-rescue:GND-power-wideband_controller_mre-rescue #PWR0104
 U 1 1 5EAEDFB7
 P 4200 1825
@@
 	2900 1375 2600 1375
 $Comp
-L wideband_controller_mre-rescue:GND-power #PWR0118
+L wideband_controller_mre-rescue:GND-power-wideband_controller_mre-rescue #PWR0118
 U 1 1 5EB4A413
 P 2900 1750
@@
 Nernst Sense Voltage Buffer
 $Comp
-L wideband_controller_mre-rescue:MCP6004-Amplifier_Operational U2
+L wideband_controller_mre-rescue:MCP6004-Amplifier_Operational-wideband_controller_mre-rescue U2
 U 2 1 5F8841DC
 P 5000 1475
@@
 $EndComp
 $Comp
-L wideband_controller_mre-rescue:MCP6004-Amplifier_Operational U2
+L wideband_controller_mre-rescue:MCP6004-Amplifier_Operational-wideband_controller_mre-rescue U2
 U 1 1 5F8980DF
 P 1925 2650
@@
 	3775 3325 3825 3325
 $Comp
-L wideband_controller_mre-rescue:MCP6004-Amplifier_Operational U2
+L wideband_controller_mre-rescue:MCP6004-Amplifier_Operational-wideband_controller_mre-rescue U2
 U 4 1 5F8B9D88
 P 1775 1375
@@
 $EndComp
 $Comp
-L wideband_controller_mre-rescue:+3.3V-power #PWR0121
+L wideband_controller_mre-rescue:+3.3V-power-wideband_controller_mre-rescue #PWR0121
 U 1 1 5F989EEA
 P 7100 2375
@@
 $EndComp
 $Comp
-L wideband_controller_mre-rescue:GND-power #PWR0122
+L wideband_controller_mre-rescue:GND-power-wideband_controller_mre-rescue #PWR0122
 U 1 1 5FE88E31
 P 5000 3800
@@
 $EndComp
 $Comp
-L wideband_controller_mre-rescue:+3.3V-power #PWR0124
+L wideband_controller_mre-rescue:+3.3V-power-wideband_controller_mre-rescue #PWR0124
 U 1 1 6014191D
 P 10025 2825
@@
 $EndComp
 $Comp
-L wideband_controller_mre-rescue:+3.3V-power #PWR0125
+L wideband_controller_mre-rescue:+3.3V-power-wideband_controller_mre-rescue #PWR0125
 U 1 1 60141F92
 P 9575 2825
@@
 $EndComp
 $Comp
-L wideband_controller_mre-rescue:GND-power #PWR0126
+L wideband_controller_mre-rescue:GND-power-wideband_controller_mre-rescue #PWR0126
 U 1 1 60142538
 P 9575 3125
@@
 $EndComp
 $Comp
-L wideband_controller_mre-rescue:GND-power #PWR0131
+L wideband_controller_mre-rescue:GND-power-wideband_controller_mre-rescue #PWR0131
 U 1 1 607B4BA6
 P 10700 4275
@@
 	7925 3750 8425 3750
 $Comp
-L wideband_controller_mre-rescue:+3.3V-power #PWR0133
+L wideband_controller_mre-rescue:+3.3V-power-wideband_controller_mre-rescue #PWR0133
 U 1 1 602BD44D
 P 1550 6725
@@
 $EndComp
 $Comp
-L wideband_controller_mre-rescue:+3.3V-power #PWR0134
+L wideband_controller_mre-rescue:+3.3V-power-wideband_controller_mre-rescue #PWR0134
 U 1 1 5FBB375A
 P 1100 6550
@@
 $EndComp
 $Comp
-L wideband_controller_mre-rescue:+3.3V-power #PWR0135
+L wideband_controller_mre-rescue:+3.3V-power-wideband_controller_mre-rescue #PWR0135
 U 1 1 5FBB1A01
 P 4025 3725
@@
 $EndComp
 $Comp
-L wideband_controller_mre-rescue:GND-power #PWR0136
+L wideband_controller_mre-rescue:GND-power-wideband_controller_mre-rescue #PWR0136
 U 1 1 5FBB1764
 P 1100 7150
@@
 $EndComp
 $Comp
-L wideband_controller_mre-rescue:MCP6004-Amplifier_Operational U2
+L wideband_controller_mre-rescue:MCP6004-Amplifier_Operational-wideband_controller_mre-rescue U2
 U 5 1 5FBAFE30
 P 1200 6850
@@
 Connection ~ 2325 3050
 $Comp
-L wideband_controller_mre-rescue:AD8603-Amplifier_Operational U3
+L wideband_controller_mre-rescue:AD8603-Amplifier_Operational-wideband_controller_mre-rescue U3
 U 1 1 5FBC4CB6
 P 4125 3425
@@
 $EndComp
 $Comp
-L wideband_controller_mre-rescue:MCP6004-Amplifier_Operational U2
+L wideband_controller_mre-rescue:MCP6004-Amplifier_Operational-wideband_controller_mre-rescue U2
 U 3 1 5F8996DF
 P 3125 4825
@@
 $EndComp
 $Comp
-L wideband_controller_mre-rescue:GND-power #PWR0138
+L wideband_controller_mre-rescue:GND-power-wideband_controller_mre-rescue #PWR0138
 U 1 1 5FBF4CD9
 P 4025 3125
@@
 $EndComp
 $Comp
-L wideband_controller_mre-rescue:GND-power #PWR0139
+L wideband_controller_mre-rescue:GND-power-wideband_controller_mre-rescue #PWR0139
 U 1 1 5FDFC1AE
 P 1975 7025
@@
 $EndComp
 $Comp
-L wideband_controller_mre-rescue:+3.3V-power #PWR0140
+L wideband_controller_mre-rescue:+3.3V-power-wideband_controller_mre-rescue #PWR0140
 U 1 1 5FDFC1B4
 P 1975 6725
@@
 $EndComp
 $Comp
-L wideband_controller_mre-rescue:GND-power #PWR0142
+L wideband_controller_mre-rescue:GND-power-wideband_controller_mre-rescue #PWR0142
 U 1 1 5FC3F94B
 P 10700 4625
@@
 UART_RX
 $Comp
-L wideband_controller_mre-rescue:GND-power #PWR0143
+L wideband_controller_mre-rescue:GND-power-wideband_controller_mre-rescue #PWR0143
 U 1 1 5FC6E3EC
 P 10250 1200
@@
 Connection ~ 7325 2425
 $Comp
-L wideband_controller_mre-rescue:GND-power #PWR0144
+L wideband_controller_mre-rescue:GND-power-wideband_controller_mre-rescue #PWR0144
 U 1 1 5FC4CC4B
 P 7425 4450
@@
 $EndComp
 $Comp
-L wideband_controller_mre-rescue:GND-power #PWR0145
+L wideband_controller_mre-rescue:GND-power-wideband_controller_mre-rescue #PWR0145
 U 1 1 5FC4C0F0
 P 7325 4450
@@
 $EndComp
 $Comp
-L wideband_controller_mre-rescue:GND-power #PWR0146
+L wideband_controller_mre-rescue:GND-power-wideband_controller_mre-rescue #PWR0146
 U 1 1 60687757
 P 6000 4250
@@
 NoConn ~ 6925 3850
 $Comp
-L wideband_controller_mre-rescue:STM32F042K6Tx-MCU_ST_STM32F0 U1
+L wideband_controller_mre-rescue:STM32F042K6Tx-MCU_ST_STM32F0-wideband_controller_mre-rescue U1
 U 1 1 5FF3B038
 P 7425 3450
@@
 	6750 2750 6400 2750
 $Comp
-L wideband_controller_mre-rescue:GND-power #PWR0147
+L wideband_controller_mre-rescue:GND-power-wideband_controller_mre-rescue #PWR0147
 U 1 1 5FE58F6B
 P 6750 3100
@@
 $EndComp
 $Comp
-L wideband_controller_mre-rescue:REF3033-Reference_Voltage U4
+L wideband_controller_mre-rescue:REF3033-Reference_Voltage-wideband_controller_mre-rescue U4
 U 1 1 5FECCFD4
 P 7875 1275
@@
 $EndComp
 $Comp
-L wideband_controller_mre-rescue:+5V-power #PWR0149
+L wideband_controller_mre-rescue:+5V-power-wideband_controller_mre-rescue #PWR0149
 U 1 1 5FECF4FF
 P 7025 800
@@
 $EndComp
 $Comp
-L wideband_controller_mre-rescue:VDDA-power #PWR0150
+L wideband_controller_mre-rescue:VDDA-power-wideband_controller_mre-rescue #PWR0150
 U 1 1 5FED060D
 P 8700 1200
@@
 $EndComp
 $Comp
-L wideband_controller_mre-rescue:VDDA-power #PWR0151
+L wideband_controller_mre-rescue:VDDA-power-wideband_controller_mre-rescue #PWR0151
 U 1 1 5FF0F5A7
 P 7425 2350
@@
 $EndComp
 $Comp
-L wideband_controller_mre-rescue:VDDA-power #PWR0152
+L wideband_controller_mre-rescue:VDDA-power-wideband_controller_mre-rescue #PWR0152
 U 1 1 5FF18494
 P 1100 875
@@
 Connection ~ 7025 875
 $Comp
-L wideband_controller_mre-rescue:GND-power #PWR0153
+L wideband_controller_mre-rescue:GND-power-wideband_controller_mre-rescue #PWR0153
 U 1 1 5FF3CC7C
 P 7025 1275
@@
 NoConn ~ 7925 3150
 $Comp
-L wideband_controller_mre-rescue:Jumper_3_Open-Jumper JP1
+L wideband_controller_mre-rescue:Jumper_3_Open-Jumper-wideband_controller_mre-rescue JP1
 U 1 1 60A55596
 P 8550 5075
@@
 $EndComp
 $Comp
-L wideband_controller_mre-rescue:+3.3V-power #PWR0155
+L wideband_controller_mre-rescue:+3.3V-power-wideband_controller_mre-rescue #PWR0155
 U 1 1 60A5820A
 P 8550 4825
@@
 SEL_1
 $Comp
-L wideband_controller_mre-rescue:Jumper_3_Open-Jumper JP2
+L wideband_controller_mre-rescue:Jumper_3_Open-Jumper-wideband_controller_mre-rescue JP2
 U 1 1 60A736F8
 P 8550 6050
@@
 $EndComp
 $Comp
-L wideband_controller_mre-rescue:+3.3V-power #PWR0157
+L wideband_controller_mre-rescue:+3.3V-power-wideband_controller_mre-rescue #PWR0157
 U 1 1 60A73704
 P 8550 5800
