File: wideband_controller_mre.kicad_pcb (KiCad board)
At the start: 2 copper layers, 80.6 x 48.4 mm, 67 parts, among them J1 TC2030, J10 Molex_Micro-Fit_3.0_43045-060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, J10 Molex_Micro-Fit_3.0_43045-061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, J2 Conn_01x06_Male, J20 Conn_02x05_Odd_Even-Connector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, J3 Conn_01x03_Male, J30 Conn_02x05_Odd_Even-Connector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, Q1 BTS3028, SW1 SW_Push, U0 wideband_MRE_R055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

Commit message: Add files via upload
Parts:
- added C42: 100nF, Capacitor_SMD:C_0603_1608Metric, F.Cu at (90.7, 157.0)
- added J15: microSD_HC_Wuerth_693072010801, Connector_Card:microSD_HC_Wuerth_693072010801, F.Cu at (100.5, 165.5)
- added J15x: MICRO-SDCARD-CONNECTOR-3300060P1, rusefi_lib:MICRO-SDCARD-CONNECTOR-3300060P1, F.Cu at (100.8, 164.8)
- moved G*** 0.64 mm to (95.5, 155.6)
- renumbered U2 to MCP6004, U1 to STM32F042K6Tx
Routing:
- net /can_fet_conn_mre_wbo2/PC11: track 0.00 -> 74.3 mm, vias 0 -> 3
- net /can_fet_conn_mre_wbo2/PC10: track 0.00 -> 69.7 mm, vias 0 -> 3
- net /can_fet_conn_mre_wbo2/PB9: track 0.00 -> 69.6 mm, vias 0 -> 3
- net /can_fet_conn_mre_wbo2/PC12: track 0.00 -> 67.2 mm, vias 0 -> 3
- net +3.3V: track 193.9 -> 249.5 mm
- net GND: track 52.6 -> 60.6 mm, vias 74 -> 82
- net /mcu_adc_mre_wbo2/nRESET: track 34.3 -> 33.3 mm
Other:
- board text added: "MRE addon board - WBO2 Controller & SDCard"
- board text added: "ver. 1.1"
- board text added: "wiring and firmware by mck1117 PCB ver.1.1 by JRD McLAREN"
- board text removed: "WIDEBAND CONTROLLER for microrusEFI"
- board text removed: "ver. 1.0"
- board text removed: "wiring and firmware by mck1117 PCB ver.1.0 by JRD McLAREN"

Commit message: Add files via upload
Connections:
- J15x pad 2: (no net) -> /can_fet_conn_mre_wbo2/PB9
- J15x pad 3: /can_fet_conn_mre_wbo2/PB9 -> /can_fet_conn_mre_wbo2/PC12
- J15x pad 4: /can_fet_conn_mre_wbo2/PC12 -> +3.3V
- J15x pad 5: +3.3V -> /can_fet_conn_mre_wbo2/PC10
- J15x pad 6: /can_fet_conn_mre_wbo2/PC10 -> GND
- J15x pad 7: GND -> /can_fet_conn_mre_wbo2/PC11
- J15x pad 8: /can_fet_conn_mre_wbo2/PC11 -> (no net)
Routing:
- net GND: track 60.6 -> 64.3 mm
- net +3.3V: track 249.5 -> 251.4 mm
- net /can_fet_conn_mre_wbo2/PC12: track 67.2 -> 65.4 mm
- net /can_fet_conn_mre_wbo2/PC10: track 69.7 -> 68.9 mm
- net /can_fet_conn_mre_wbo2/PB9: track 69.6 -> 68.8 mm
- net /can_fet_conn_mre_wbo2/PC11: track 74.3 -> 73.5 mm

Commit message: Add files via upload
Parts:
- added C25: 10nF, Capacitor_SMD:C_0603_1608Metric, F.Cu at (80.0, 135.0)
- added C26: 100nF, Capacitor_SMD:C_0603_1608Metric, F.Cu at (83.1, 135.0)
- added J1: PinHeader_1x01_P2.54mm_Vertical, Connector_PinHeader_2.54mm:PinHeader_1x01_P2.54mm_Vertical, F.Cu at (151.6, 129.0)
- added J40: CONN_Molex, Connector_Molex:Molex_Micro-Fit_3.0_43045-0200_2x01_P3.00mm_Horizontal, F.Cu at (84.5, 129.9)
- added J40x: Molex_Micro-Fit_3.0_43045-0212_2x01_P3.00mm_Vertical, Connector_Molex:Molex_Micro-Fit_3.0_43045-0212_2x01_P3.00mm_Vertical, F.Cu at (84.5, 129.9)
- added J41: CONN_Sparkfun, rusefi_lib:tcpl_PCC-SMP, F.Cu at (23.7, 132.8)
- added MAX31855: MAX31855KASA, Package_SO:SO-8_5.3x6.2mm_P1.27mm, F.Cu at (80.0, 140.9)
- moved C42 13.2 mm to (91.2, 170.2), turned to 270 degrees
- moved C24 5.01 mm to (86.7, 143.2)
- moved C23 5.00 mm to (90.3, 143.2)
- moved TJA1051T 4.11 mm to (88.4, 136.7), turned to 180 degrees
- moved SW1 1.10 mm to (97.4, 137.2)
- renumbered STM32F042K6Tx to STM32F042K6T, U5 to TJA1051T
Routing:
- net /can_fet_conn_mre_wbo2/PA15: track 0.00 -> 77.7 mm, vias 0 -> 2
- net /can_fet_conn_mre_wbo2/PC10: track 68.9 -> 98.4 mm
- net /can_fet_conn_mre_wbo2/PC11: track 73.5 -> 95.7 mm
- net /can_fet_conn_mre_wbo2/TCPL-: track 0.00 -> 12.0 mm
- net /can_fet_conn_mre_wbo2/TCPL+: track 0.00 -> 9.98 mm
- net CAN_RX: track 24.8 -> 15.0 mm
- net +5V: track 144.1 -> 139.3 mm
- net +3.3V: track 251.4 -> 255.6 mm
- net /can_fet_conn_mre_wbo2/12V_MREL: track 7.27 -> 11.1 mm
- net /can_fet_conn_mre_wbo2/CAN_H: track 6.57 -> 9.96 mm, vias 0 -> 1
- net /can_fet_conn_mre_wbo2/CAN_L: track 6.78 -> 9.38 mm, vias 0 -> 1
- net GND: track 64.3 -> 62.5 mm, vias 82 -> 86
- net /mcu_adc_mre_wbo2/Boot0: track 27.0 -> 25.6 mm
- net CAN_TX: track 19.1 -> 17.8 mm
Other:
- board text added: "H"
- board text added: "JP1, JP2: low, low = idx 2 low, float = idx 0 low, high = idx 3 float, low = idx 4 float, float = read index from flash cfg float, high = idx 1 high, low = idx 5 high, float = idx 6 high, high = idx 7"
- board text added: "K - Thermocouple"
- board text added: "L"
- board text added: "TCPL +"
- board text added: "TCPL -"
- board text added: "WBO2 controller by mck1117 PCB ver.1.2 by JRD McLAREN"
- board text added: "ver. 1.2"
- board text removed: "SEL_1, SEL_2: low, low = idx 2 low, float = idx 0 low, high = idx 3 float, low = idx 4 float, float = read index from flash cfg float, high = idx 1 high, low = idx 5 high, float = idx 6 high, high = idx 7"
- board text removed: "ver. 1.1"
- board text removed: "wiring and firmware by mck1117 PCB ver.1.1 by JRD McLAREN"
