File: wideband_controller_mre.kicad_pcb (KiCad board)
At the start: 2 copper layers, 80.6 x 48.4 mm, 77 parts, among them J1 PinHeader_1x01_P2.54mm_Vertic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, J1 TC2030, J10 Molex_Micro-Fit_3.0_43045-060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, J10 Molex_Micro-Fit_3.0_43045-061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, J15 microSD_HC_Wuerth_693072010801, J15x MICRO-SDCARD-CONNECTOR-330006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, J2 Conn_01x06_Male, J20 Conn_02x05_Odd_Even-Connector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, J3 Conn_01x03_Male, J30 Conn_02x05_Odd_Even-Connector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

Commit message: Add files via upload
Parts:
- renumbered STM32F042K6T to U1, MCP6004 to U2, TJA1051T to U5, MAX31855 to U6
Other:
- board text added: "MAX31855"
- board text added: "MCP6004"
- board text added: "STM32F042K6T"
- board text added: "TJA1051T"
Changed lines of the file:
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@@
   (general
     (thickness 1.6)
-    (drawings 51)
+    (drawings 55)
     (tracks 821)
     (zones 0)
@@
     (tags "SOIC 1.27")
     (attr smd)
-    (fp_text reference MAX31855 (at 0.1 0 180) (layer F.SilkS)
+    (fp_text reference U6 (at 0.1 0 180) (layer F.SilkS) hide
       (effects (font (size 0.75 0.75) (thickness 0.125)))
     )
@@
     (tags "SOIC SO")
     (attr smd)
-    (fp_text reference TJA1051T (at 0 0 270) (layer F.SilkS)
+    (fp_text reference U5 (at 0 0 270) (layer F.SilkS) hide
       (effects (font (size 0.75 0.75) (thickness 0.125)))
     )
@@
     (tags "SSOP 0.65")
     (attr smd)
-    (fp_text reference MCP6004 (at -0.1 0) (layer F.SilkS)
+    (fp_text reference U2 (at -0.1 0) (layer F.SilkS) hide
       (effects (font (size 0.7 0.7) (thickness 0.15)))
     )
@@
     (tags "LQFP QFP")
     (attr smd)
-    (fp_text reference STM32F042K6T (at 0 -5.7 180) (layer F.SilkS)
+    (fp_text reference U1 (at 0 0.1 180) (layer F.SilkS)
       (effects (font (size 0.8 0.8) (thickness 0.15)))
     )
@@
     )
   )
+  (gr_text MAX31855 (at 80.1 141) (layer F.SilkS)
+    (effects (font (size 0.5 0.5) (thickness 0.125)))
+  )
+  (gr_text TJA1051T (at 88.3 136.7 90) (layer F.SilkS)
+    (effects (font (size 0.5 0.5) (thickness 0.125)))
+  )
+  (gr_text MCP6004 (at 123 135.2) (layer F.SilkS)
+    (effects (font (size 0.7 0.7) (thickness 0.15)))
+  )
+  (gr_text STM32F042K6T (at 109.2 142.2) (layer F.SilkS)
+    (effects (font (size 0.75 0.75) (thickness 0.15)))
+  )
   (gr_text "K - Thermocouple" (at 82.7 132.9) (layer B.SilkS)

Commit message: Add files via upload
Other:
- board text added: "MRE addon board - WBO2 & EGT & SDCard"
- board text removed: "MRE addon board - WBO2 Controller & SDCard"
Changed lines of the file:
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@@
     (effects (font (size 1 1) (thickness 0.25)))
   )
-  (gr_text "MRE addon board - WBO2 Controller & SDCard" (at 115.5 173) (layer F.SilkS)
+  (gr_text "MRE addon board - WBO2 & EGT & SDCard" (at 115.5 173) (layer F.SilkS)
     (effects (font (size 1.5 1.5) (thickness 0.3)))
   )

Commit message: Add files via upload
Parts:
- removed the J1 at (151.6, 129.0)
- added C21: 100nF, Capacitor_SMD:C_0603_1608Metric, F.Cu at (92.1, 132.4)
- added J21: Soldering PAD for 12V_MREL, Connector_PinHeader_2.54mm:PinHeader_1x01_P2.54mm_Vertical, F.Cu at (151.6, 129.0)
- moved J3 0.10 mm to (94.7, 133.2)
- moved C12 0.10 mm to (103.1, 131.0)
Routing:
- net +5V: track 139.3 -> 145.2 mm
Changed lines of the file:
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@@
     (thickness 1.6)
     (drawings 55)
-    (tracks 821)
+    (tracks 830)
     (zones 0)
-    (modules 77)
+    (modules 78)
     (nets 73)
   )
@@
     (descr "Through hole straight pin header, 1x01, 2.54mm pitch, single row")
     (tags "Through hole pin header THT 1x01 2.54mm single row")
-    (fp_text reference J1 (at 0 -2.33) (layer F.SilkS)
+    (fp_text reference J21 (at 0 -2.33) (layer F.SilkS)
       (effects (font (size 1 1) (thickness 0.15)))
     )
-    (fp_text value PinHeader_1x01_P2.54mm_Vertical (at 0 2.33) (layer F.Fab)
+    (fp_text value "Soldering PAD for 12V_MREL" (at 0 2.33) (layer F.Fab)
       (effects (font (size 1 1) (thickness 0.15)))
     )
@@
     )
   )
+  (module Capacitor_SMD:C_0603_1608Metric (layer F.Cu)
+    (at 92.1 132.4 90)
+    (descr "Capacitor SMD 0603 (1608 Metric), square (rectangular) end terminal, IPC_7351 nominal, (Body size source: http://www.tortai-tech.com/upload/download/2011102023233369053.pdf), generated with kicad-footprint-generator")
+    (tags capacitor)
+    (attr smd)
+    (fp_text reference C21 (at 0 -1.43 90) (layer F.SilkS)
+      (effects (font (size 1 1) (thickness 0.15)))
+    )
+    (fp_text value 100nF (at 0 1.43 90) (layer F.Fab)
+      (effects (font (size 1 1) (thickness 0.15)))
+    )
+    (fp_text user %R (at 0 0 90) (layer F.Fab)
+      (effects (font (size 0.4 0.4) (thickness 0.06)))
+    )
+    (fp_line (start 1.48 0.73) (end -1.48 0.73) (layer F.CrtYd) (width 0.05))
+    (fp_line (start 1.48 -0.73) (end 1.48 0.73) (layer F.CrtYd) (width 0.05))
+    (fp_line (start -1.48 -0.73) (end 1.48 -0.73) (layer F.CrtYd) (width 0.05))
+    (fp_line (start -1.48 0.73) (end -1.48 -0.73) (layer F.CrtYd) (width 0.05))
+    (fp_line (start -0.162779 0.51) (end 0.162779 0.51) (layer F.SilkS) (width 0.12))
+    (fp_line (start -0.162779 -0.51) (end 0.162779 -0.51) (layer F.SilkS) (width 0.12))
+    (fp_line (start 0.8 0.4) (end -0.8 0.4) (layer F.Fab) (width 0.1))
+    (fp_line (start 0.8 -0.4) (end 0.8 0.4) (layer F.Fab) (width 0.1))
+    (fp_line (start -0.8 -0.4) (end 0.8 -0.4) (layer F.Fab) (width 0.1))
+    (fp_line (start -0.8 0.4) (end -0.8 -0.4) (layer F.Fab) (width 0.1))
+    (pad 2 smd roundrect (at 0.7875 0 90) (size 0.875 0.95) (layers F.Cu F.Paste F.Mask) (roundrect_rratio 0.25)
+      (net 12 +5V))
+    (pad 1 smd roundrect (at -0.7875 0 90) (size 0.875 0.95) (layers F.Cu F.Paste F.Mask) (roundrect_rratio 0.25)
+      (net 1 GND))
+    (model ${KISYS3DMOD}/Capacitor_SMD.3dshapes/C_0603_1608Metric.wrl
+      (at (xyz 0 0 0))
+      (scale (xyz 1 1 1))
+      (rotate (xyz 0 0 0))
+    )
+  )
   (module Connector_Molex:Molex_Micro-Fit_3.0_43045-0212_2x01_P3.00mm_Vertical (layer F.Cu)
     (at 84.5 129.9 90)
@@
   )
   (module Connector_PinHeader_2.54mm:PinHeader_1x03_P2.54mm_Vertical (layer F.Cu)
-    (at 94.6 133.2 90)
+    (at 94.7 133.2 90)
     (descr "Through hole straight pin header, 1x03, 2.54mm pitch, single row")
     (tags "Through hole pin header THT 1x03 2.54mm single row")
@@
   )
   (module Capacitor_SMD:C_0603_1608Metric (layer F.Cu)
-    (at 103 131)
+    (at 103.1 131)
     (descr "Capacitor SMD 0603 (1608 Metric), square (rectangular) end terminal, IPC_7351 nominal, (Body size source: http://www.tortai-tech.com/upload/download/2011102023233369053.pdf), generated with kicad-footprint-generator")
     (tags capacitor)
@@
   (segment (start 88.3 134.8) (end 89.8 134.8) (width 0.5) (layer B.Cu) (net 8))
   (segment (start 94.144999 139.155001) (end 89.9 134.9) (width 0.5) (layer B.Cu) (net 8))
-  (segment (start 89 134.1) (end 88.3 134.8) (width 0.3) (layer F.Cu) (net 8))
-  (segment (start 90.865 134.1) (end 89 134.1) (width 0.3) (layer F.Cu) (net 8))
-  (segment (start 95.33 129.635) (end 90.865 134.1) (width 0.3) (layer F.Cu) (net 8))
+  (segment (start 88.699999 134.400001) (end 88.3 134.8) (width 0.3) (layer F.Cu) (net 8))
+  (segment (start 89.290001 133.809999) (end 88.699999 134.400001) (width 0.3) (layer F.Cu) (net 8))
+  (segment (start 89.290001 133.143149) (end 89.290001 133.809999) (width 0.3) (layer F.Cu) (net 8))
+  (segment (start 94.936301 130.028699) (end 92.404451 130.028699) (width 0.3) (layer F.Cu) (net 8))
+  (segment (start 92.404451 130.028699) (end 89.290001 133.143149) (width 0.3) (layer F.Cu) (net 8))
+  (segment (start 95.33 129.635) (end 94.936301 130.028699) (width 0.3) (layer F.Cu) (net 8))
   (via (at 124.4 129.8) (size 0.6) (drill 0.3) (layers F.Cu B.Cu) (net 9))
   (segment (start 124.4 128.9875) (end 124.425 128.9875) (width 0.25) (layer F.Cu) (net 9))
@@
   (segment (start 89.265 136.065) (end 89.25 136.05) (width 0.5) (layer F.Cu) (net 12))
   (segment (start 90.875 136.065) (end 89.265 136.065) (width 0.5) (layer F.Cu) (net 12))
+  (segment (start 89.25 135.484315) (end 89.25 136.05) (width 0.3) (layer F.Cu) (net 12))
+  (segment (start 89.790011 134.197865) (end 89.25 134.737876) (width 0.3) (layer F.Cu) (net 12))
+  (segment (start 89.790011 133.447489) (end 89.790011 134.197865) (width 0.3) (layer F.Cu) (net 12))
+  (segment (start 89.25 134.737876) (end 89.25 135.484315) (width 0.3) (layer F.Cu) (net 12))
+  (segment (start 91.625 131.6125) (end 89.790011 133.447489) (width 0.3) (layer F.Cu) (net 12))
+  (segment (start 92.1 131.6125) (end 91.625 131.6125) (width 0.3) (layer F.Cu) (net 12))
   (via (at 87.2 137.3) (size 0.6) (drill 0.3) (layers F.Cu B.Cu) (net 13))
   (segment (start 90.9875 140.3987) (end 91.3606 140.7718) (width 0.3) (layer F.Cu) (net 13))

Commit message: Add files via upload
Parts:
- added U3: AD8628, Package_SO:SO-8_3.9x4.9mm_P1.27mm, F.Cu at (122.7, 147.3)
- moved R16 6.38 mm to (118.8, 150.8), turned to 0 degrees
- moved C11 4.67 mm to (118.0, 145.5), turned to 90 degrees
- moved R14 3.58 mm to (127.2, 142.4), turned to 90 degrees
- moved R18 2.14 mm to (118.0, 148.5), turned to 90 degrees
- moved R17 1.42 mm to (127.7, 147.3)
- moved R17 1.39 mm to (127.7, 147.3)
- moved R13 1.12 mm to (126.5, 150.8)
- moved U3 0.58 mm to (122.7, 147.6)
- moved C6 0.55 mm to (122.8, 150.8)
- moved C5 0.20 mm to (128.4, 139.0)
- moved R7 0.20 mm to (126.8, 139.0)
- moved R8 0.20 mm to (119.2, 139.0)
Routing:
- net GND: track 62.5 -> 79.2 mm, vias 86 -> 83
- net Net-(R16-Pad1): track 8.14 -> 17.7 mm
- net Net-(R14-Pad1): track 8.81 -> 17.4 mm
- net Net-(R13-Pad1): track 7.87 -> 14.1 mm
- net LSU_Rtrim: track 32.0 -> 34.0 mm
- net LSU_Ip: track 22.8 -> 21.8 mm
- net heater_pwm: track 48.2 -> 47.6 mm
- net /mcu_adc_mre_wbo2/Ip_sense: track 20.6 -> 20.0 mm
- net +3.3V: track 256.0 -> 255.5 mm, vias 5 -> 7
Other:
- board text added: "AD8628"
- board text added: "JP1, JP2: low, low = idx 2 low, float = idx 0 low, high = idx 3 float, low = idx 4 float, high = idx 1 high, low = idx 5 high, float = idx 6 high, high = idx 7 float, float = read index from flash cfg"
- board text added: "WBO2 controller by mck1117 PCB ver.1.3 by JRD McLAREN"
- board text added: "ver. 1.3"
- board text removed: "JP1, JP2: low, low = idx 2 low, float = idx 0 low, high = idx 3 float, low = idx 4 float, float = read index from flash cfg float, high = idx 1 high, low = idx 5 high, float = idx 6 high, high = idx 7"
- board text removed: "WBO2 controller by mck1117 PCB ver.1.2 by JRD McLAREN"
- board text removed: "ver. 1.2"

Commit message: Add files via upload
Parts:
- added D1: RED, LED_SMD:LED_0603_1608Metric, B.Cu at (136.8, 156.6)
- added D2: GREEN, LED_SMD:LED_0603_1608Metric, B.Cu at (111.3, 144.8)
- added D3: BLUE, LED_SMD:LED_0603_1608Metric, B.Cu at (111.3, 146.3)
- F1: footprint Resistor_SMD:R_1206_3216Metric -> Resistor_SMD:R_2816_7142Metric
- moved J21 0.80 mm to (151.6, 128.2)
- moved F1 0.07 mm to (151.7, 134.3)
Routing:
- net GND: track 79.2 -> 81.4 mm, vias 83 -> 84
- net /can_fet_conn_mre_wbo2/LSU_Heater+: track 14.9 -> 13.1 mm
- net +5V: track 145.2 -> 143.7 mm
- net /can_fet_conn_mre_wbo2/12V_MREL: track 11.1 -> 10.2 mm
- net Net-(D1-Pad2): track 2.25 -> 2.88 mm, vias 0 -> 1
- net /mcu_adc_mre_wbo2/Nernst_esr_drive: track 30.3 -> 30.8 mm
- net /mcu_adc_mre_wbo2/LED_GREEN: track 4.86 -> 5.37 mm, vias 0 -> 1
- net /mcu_adc_mre_wbo2/LED_BLUE: track 6.69 -> 7.20 mm, vias 0 -> 1
- net Net-(D3-Pad1): track 1.52 -> 2.04 mm, vias 0 -> 1
- net Net-(D2-Pad1): track 1.57 -> 2.08 mm, vias 0 -> 1
Other:
- board text added: "JP1, JP2: low, low = idx 2 low, float = idx 0 low, high = idx 3 float, low = idx 4 float, high = idx 1 high, low = idx 5 high, float = idx 6 high, high = idx 7 float, float = read idx from flash"
- board text removed: "JP1, JP2: low, low = idx 2 low, float = idx 0 low, high = idx 3 float, low = idx 4 float, high = idx 1 high, low = idx 5 high, float = idx 6 high, high = idx 7 float, float = read index from flash cfg"
